File: TRswitch/TRswitch.sch (KiCad schematic (older format))
At the start: 21 parts

Commit message: Work on text and fig2
Parts:
- removed C? (x2): 0.1u, symbol C
- added C? (x11): 0.1u, symbol C
- added R?: 2K2, symbol R
- L? (x4): value INDUCTOR -> 100 uH
Connections:
- wire segments 21 -> 31
Other:
- moved on the sheet: C?, L?, R?
Changed lines of the file:
@@
-EESchema Schematic File Version 2  date Wed 08 Jan 2014 16:44:26 NZDT
+EESchema Schematic File Version 2  date Thu 06 Feb 2014 08:15:03 NZDT
 LIBS:power
 LIBS:device
@@
 LIBS:contrib
 LIBS:valves
+LIBS:TRswitch-cache
 EELAYER 25  0
 EELAYER END
@@
 Sheet 1 1
 Title ""
-Date "8 jan 2014"
+Date "5 feb 2014"
 Rev ""
 Comp ""
@@
 Comment4 ""
 $EndDescr
-Connection ~ 1700 2350
-Connection ~ 4950 2500
+Wire Wire Line
+	3750 2500 4000 2500
+Wire Wire Line
+	3750 2500 3750 2600
+Connection ~ 3000 2150
+Wire Wire Line
+	2800 2150 3200 2150
+Wire Wire Line
+	3000 1150 3000 1350
+Wire Wire Line
+	3200 1350 2800 1350
+Connection ~ 3000 1350
+Connection ~ 1100 2550
+Wire Wire Line
+	1100 2550 1300 2550
+Wire Wire Line
+	1100 2900 1100 2750
+Connection ~ 1100 2750
+Connection ~ 2100 2350
+Wire Wire Line
+	2100 2550 2100 2150
+Connection ~ 5900 2550
+Wire Wire Line
+	5900 2550 5750 2550
+Wire Wire Line
+	4950 2550 4950 2150
+Connection ~ 5900 2750
 Connection ~ 4950 2350
-Connection ~ 1700 2500
-Wire Wire Line
-	1700 2650 1700 2500
 Wire Wire Line
 	4500 3000 4500 2850
@@
 	3900 1200 3900 1100
 Wire Wire Line
-	3000 1850 3000 1150
-Wire Wire Line
 	2200 3550 2200 3600
 Connection ~ 3000 2350
 Wire Wire Line
-	3000 2250 3000 2350
+	3000 2350 3000 2150
 Wire Wire Line
 	2600 2350 3600 2350
@@
 	3600 2350 3600 2200
 Wire Wire Line
-	4000 2350 4000 2450
+	4000 2500 4000 2350
 Wire Wire Line
 	4500 2850 4850 2850
@@
 	2200 2350 2100 2350
 Wire Wire Line
-	4000 3600 4000 3550
-Wire Wire Line
-	4400 2350 4550 2350
+	4400 2350 4950 2350
 Connection ~ 4500 2350
 Wire Wire Line
@@
 Connection ~ 4250 3600
 Wire Wire Line
-	4900 1100 3600 1100
+	3600 1100 4900 1100
 Connection ~ 4700 1100
 Wire Wire Line
-	4950 2650 4950 2500
+	5900 2900 5900 2750
+Wire Wire Line
+	5750 2550 5750 2150
+Wire Wire Line
+	1300 2550 1300 2150
+Wire Wire Line
+	3750 3100 4000 3100
+$Comp
+L R R?
+U 1 1 52F28CF7
+P 3750 2850
+F 0 "R?" V 3830 2850 50  0000 C CNN
+F 1 "2K2" V 3750 2850 50  0000 C CNN
+	1    3750 2850
+	1    0    0    -1
+$EndComp
+$Comp
+L C C?
+U 1 1 52F28C41
+P 2800 1550
+F 0 "C?" H 2850 1650 50  0000 L CNN
+F 1 "0.1u" H 2850 1450 50  0000 L CNN
+	1    2800 1550
+	-1   0    0    1
+$EndComp
+$Comp
+L C C?
+U 1 1 52F28C40
+P 3200 1950
+F 0 "C?" H 3250 2050 50  0000 L CNN
+F 1 "0.1u" H 3250 1850 50  0000 L CNN
+	1    3200 1950
+	-1   0    0    1
+$EndComp
+$Comp
+L C C?
+U 1 1 52F28C3F
+P 3200 1550
+F 0 "C?" H 3250 1650 50  0000 L CNN
+F 1 "0.1u" H 3250 1450 50  0000 L CNN
+	1    3200 1550
+	-1   0    0    1
+$EndComp
+$Comp
+L C C?
+U 1 1 52F28C3E
+P 2800 1950
+F 0 "C?" H 2850 2050 50  0000 L CNN
+F 1 "0.1u" H 2850 1850 50  0000 L CNN
+	1    2800 1950
+	-1   0    0    1
+$EndComp
+$Comp
+L GND #PWR?
+U 1 1 52F28BBC
+P 1100 2900
+F 0 "#PWR?" H 1100 2900 30  0001 C CNN
+F 1 "GND" H 1100 2830 30  0001 C CNN
+	1    1100 2900
+	1    0    0    -1
+$EndComp
+$Comp
+L C C?
+U 1 1 52F28B0A
+P 1500 2150
+F 0 "C?" H 1550 2250 50  0000 L CNN
+F 1 "0.1u" H 1550 2050 50  0000 L CNN
+	1    1500 2150
+	0    -1   -1   0
+$EndComp
+$Comp
+L C C?
+U 1 1 52F28B09
+P 1900 2550
+F 0 "C?" H 1950 2650 50  0000 L CNN
+F 1 "0.1u" H 1950 2450 50  0000 L CNN
+	1    1900 2550
+	0    -1   -1   0
+$EndComp
+$Comp
+L C C?
+U 1 1 52F28B08
+P 1500 2550
+F 0 "C?" H 1550 2650 50  0000 L CNN
+F 1 "0.1u" H 1550 2450 50  0000 L CNN
+	1    1500 2550
+	0    -1   -1   0
+$EndComp
+$Comp
+L C C?
+U 1 1 52F28B07
+P 1900 2150
+F 0 "C?" H 1950 2250 50  0000 L CNN
+F 1 "0.1u" H 1950 2050 50  0000 L CNN
+	1    1900 2150
+	0    -1   -1   0
+$EndComp
+$Comp
+L C C?
+U 1 1 52F28AB5
+P 5550 2150
+F 0 "C?" H 5600 2250 50  0000 L CNN
+F 1 "0.1u" H 5600 2050 50  0000 L CNN
+	1    5550 2150
+	0    -1   -1   0
+$EndComp
+$Comp
+L C C?
+U 1 1 52F28A3B
+P 5150 2550
+F 0 "C?" H 5200 2650 50  0000 L CNN
+F 1 "0.1u" H 5200 2450 50  0000 L CNN
+	1    5150 2550
+	0    -1   -1   0
+$EndComp
+$Comp
+L C C?
+U 1 1 52F28A2E
+P 5550 2550
+F 0 "C?" H 5600 2650 50  0000 L CNN
+F 1 "0.1u" H 5600 2450 50  0000 L CNN
+	1    5550 2550
+	0    -1   -1   0
+$EndComp
 $Comp
 L GND #PWR?
 U 1 1 52CCC663
-P 4950 2650
-F 0 "#PWR?" H 4950 2650 30  0001 C CNN
-F 1 "GND" H 4950 2580 30  0001 C CNN
-	1    4950 2650
-	1    0    0    -1
-$EndComp
-$Comp
-L GND #PWR?
-U 1 1 52CCC656
-P 1700 2650
-F 0 "#PWR?" H 1700 2650 30  0001 C CNN
-F 1 "GND" H 1700 2580 30  0001 C CNN
-	1    1700 2650
+P 5900 2900
+F 0 "#PWR?" H 5900 2900 30  0001 C CNN
+F 1 "GND" H 5900 2830 30  0001 C CNN
+	1    5900 2900
 	1    0    0    -1
 $EndComp
@@
 L C C?
 U 1 1 52CCBEF5
-P 4750 2350
-F 0 "C?" H 4800 2450 50  0000 L CNN
-F 1 "0.1u" H 4800 2250 50  0000 L CNN
-	1    4750 2350
-	0    -1   -1   0
-$EndComp
-$Comp
-L C C?
-U 1 1 52CCBE49
-P 1900 2350
-F 0 "C?" H 1950 2450 50  0000 L CNN
-F 1 "0.1u" H 1950 2250 50  0000 L CNN
-	1    1900 2350
-	0    -1   -1   0
-$EndComp
-$Comp
-L C C?
-U 1 1 52CCBD46
-P 3000 2050
-F 0 "C?" H 3050 2150 50  0000 L CNN
-F 1 "0.1u" H 3050 1950 50  0000 L CNN
-	1    3000 2050
-	1    0    0    -1
+P 5150 2150
+F 0 "C?" H 5200 2250 50  0000 L CNN
+F 1 "0.1u" H 5200 2050 50  0000 L CNN
+	1    5150 2150
+	0    -1   -1   0
 $EndComp
 $Comp
@@
 P 2200 2750
 F 0 "L?" V 2150 2750 40  0000 C CNN
-F 1 "INDUCTOR" V 2300 2750 40  0000 C CNN
+F 1 "100 uH" V 2300 2750 40  0000 C CNN
 	1    2200 2750
 	-1   0    0    -1
@@
 	1    0    0    1
 $EndComp
-Text Notes 1300 2450 0    60   ~ 0
+Text Notes 900  2450 0    60   ~ 0
 TX out
 $Comp
@@
 U 1 1 52CC8278
 P 4200 2350
-F 0 "D?" H 4200 2450 40  0000 C CNN
+F 0 "D?" H 4200 2150 40  0000 C CNN
 F 1 "1N4007" H 4200 2250 40  0000 C CNN
 	1    4200 2350
@@
 U 1 1 52CC8277
 P 3800 2350
-F 0 "D?" H 3800 2450 40  0000 C CNN
+F 0 "D?" H 3800 2150 40  0000 C CNN
 F 1 "1N4007" H 3800 2250 40  0000 C CNN
 	1    3800 2350
@@
 L INDUCTOR L?
 U 1 1 52CC8276
-P 4000 2750
-F 0 "L?" V 3950 2750 40  0000 C CNN
-F 1 "INDUCTOR" V 4100 2750 40  0000 C CNN
-	1    4000 2750
+P 4000 2800
+F 0 "L?" V 3950 2800 40  0000 C CNN
+F 1 "100 uH" V 4100 2800 40  0000 C CNN
+	1    4000 2800
 	1    0    0    -1
 $EndComp
@@
 P 4400 1900
 F 0 "L?" V 4350 1900 40  0000 C CNN
-F 1 "INDUCTOR" V 4500 1900 40  0000 C CNN
+F 1 "100 uH" V 4500 1900 40  0000 C CNN
 	1    4400 1900
 	1    0    0    -1
@@
 P 3600 1900
 F 0 "L?" V 3550 1900 40  0000 C CNN
-F 1 "INDUCTOR" V 3700 1900 40  0000 C CNN
+F 1 "100 uH" V 3700 1900 40  0000 C CNN
 	1    3600 1900
 	1    0    0    -1
@@
 L R R?
 U 1 1 52CC8272
-P 4000 3300
-F 0 "R?" V 4080 3300 50  0000 C CNN
-F 1 "150R" V 4000 3300 50  0000 C CNN
-	1    4000 3300
-	1    0    0    -1
-$EndComp
-Text Notes 5050 2450 0    60   ~ 0
+P 4000 3350
+F 0 "R?" V 4080 3350 50  0000 C CNN
+F 1 "150R" V 4000 3350 50  0000 C CNN
+	1    4000 3350
+	1    0    0    -1
+$EndComp
+Text Notes 5800 2450 0    60   ~ 0
 RX in
 $Comp

Commit message: Changes to TRswitch schematic
Parts:
- added Q? (x2): PNP, symbol PNP
- added Q? (x4): NPN, symbol NPN
- added R? (x5): 2K2, symbol R
- added R?: 4K7, symbol R
- added R? (x2): 15K, symbol R
Connections:
- net labels added: +12V
- wire segments 31 -> 72

Commit message: More work on schematic
Parts:
- removed Q? (x2): PNP, symbol PNP
- removed Q? (x4): NPN, symbol NPN
- removed R?: 4K7, symbol R
- removed R?: 2K2, symbol R
- added C16: 0.1uF, symbol C
- added C19: 100uF, symbol CP
- added D1: DIODESCH, symbol DIODESCH
- added D3: DIODE, symbol DIODE
- added Q1, Q2: PN100, TO92-EBC, symbol BC237
- added Q3, Q5: BD140, symbol BC307
- added Q4, Q6: BD139, TO92-EBC, symbol BC237
- added R13, R4: 22K, symbol R
- D2, D4, D5, D6: renamed from D?; value 1N4007 -> GP10Y
- R11, R6: renamed from R?; value 3R3 -> 2R2
- R9: renamed from R?; value 150R -> 100R
- gave numbers to parts that had none: 30
Connections:
- wire segments 72 -> 98
Other:
- moved on the sheet: C1, C10, C11, C12, C13, C14, C15, C17, C18, C2, C3, C4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

Commit message: More work on schematic
Parts:
- removed D1: DIODESCH, symbol DIODESCH
- added C1, C10, C14, C17, C2, C26, C3: 0.1u, symbol C
- added D1: 1N4148, symbol DIODE
- added D4: GP10Y, symbol DIODE
- added P1: Tx out, symbol CONNECTOR
- added P2: Antenna, symbol CONNECTOR
- added P3: Rx in, symbol CONNECTOR
- added R5, R7: 1M, symbol R
- C22: renamed from C16; value 0.1uF -> 0.1u
- D2: renamed from D3; value DIODE -> 1N4148
- R1, R2: value 15K -> 10K
- renumbered C18 to C11, C15 to C12, C5 to C13, C6 to C15, C7 to C16, C8 to C18, C9 to C19, C10 to C20, C11 to C21, C12 to C23, C19 to C24, C13 to C25, C14 to C4, C1 to C5, C2 to C6, C17 to C7, C3 to C8, C4 to C9, D2 to D3, D4 to D5, D5 to D6, D6 to D7, R6 to R10, R7 to R11, R9 to R12, R11 to R15, R12 to R16, R4 to R3, R5 to R4, R3 to R6, R10 to R9
Connections:
- wire segments 98 -> 73
Other:
- note removed: "Antenna"
- note removed: "RX in"
- note removed: "TX out"
- moved on the sheet: C11, C12, C13, C15, C16, C18, C19, C20, C21, C23, C25, C4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

Commit message: Started on PCB Layout
Parts:
- removed P1: Tx out, symbol CONNECTOR
- removed P2: Antenna, symbol CONNECTOR
- removed P3: Rx in, symbol CONNECTOR
- added Antenna1, Eth1, Eth2, Eth3, Rx1, Tx1: CONN_1, symbol CONN_1
- added C10, C21, C23, C27: 0.1u, symbol C
- added P1: Tx/Rx, symbol CONN_2
- renumbered C10 to C11, C11 to C12, C12 to C13, C13 to C14, C14 to C15, C15 to C16, C16 to C17, C17 to C18, C18 to C19, C19 to C20, C20 to C22, C21 to C24, C22 to C25, C23 to C26, C24 to C28, C25 to C29, C26 to C30
Connections:
- wire segments 73 -> 76
Other:
- note added: "Drive from open collector\nwith Tx Low, Rx open."
- moved on the sheet: C22, C26, R10, R11, R15

Commit message: More work on PCB
Parts:
- added +12v1, Bias-1, Bias-2, Bias_1, Bias_2: CONN_1, symbol CONN_1
Connections:
- net GND: no longer C25.2, C28.2, D2.2 (K), P1.2 (PM), Q1.E, Q4.E, Q6.E
- net at D4.2 (K), D5.1 (A), L2.2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: now also C13.1, C17.1, C20.1
- net +12V: no longer names the net of C25.1, C28.1, Q3.E, Q5.E, R1.1, R13.2, R2.1, R3.1
- net +12V: now also +12v1.1
- net Bias1: no longer names the net of C22.1, C26.1, R10.1, R15.1
- net Bias1: now also Bias-1.1; no longer Q5.C, Q6.C, R8.2
- net Bias2: no longer names the net of C14.1, C24.1, R12.2, R16.1, R6.1
- net Bias2: now also Bias-2.1; no longer Q3.C, Q4.C, R9.2
- new net: Bias_1.1, Q5.C, Q6.C, R8.2
- new net: Bias_2.1, Q3.C, Q4.C, R9.2
- new net AGND: C25.2, C28.2, D2.2 (K), P1.2 (PM), Q1.E, Q4.E, Q6.E

Commit message: Reduced size of PCB
Parts:
- removed C26: 0.1u, symbol C
Changed lines of the file:
@@
-EESchema Schematic File Version 2  date Wed 19 Feb 2014 15:03:23 NZDT
+EESchema Schematic File Version 2  date Thu 20 Feb 2014 23:05:03 NZDT
 LIBS:power
 LIBS:device
@@
 Sheet 1 1
 Title ""
-Date "19 feb 2014"
+Date "20 feb 2014"
 Rev ""
 Comp ""
@@
 Comment4 ""
 $EndDescr
+Wire Wire Line
+	5300 1150 6600 1150
+Connection ~ 11500 4850
+Connection ~ 5300 1750
+Connection ~ 6100 1750
+Connection ~ 3300 2500
+Connection ~ 3300 3800
+Connection ~ 3250 5350
+Connection ~ 5750 5350
+Connection ~ 3650 4850
+Connection ~ 3650 7000
+Wire Wire Line
+	6800 2500 6950 2500
+Wire Wire Line
+	4700 950  4700 1100
+Wire Wire Line
+	6100 1650 6100 1750
+Wire Wire Line
+	6100 1750 6400 1750
+Wire Wire Line
+	6400 2500 6100 2500
+Connection ~ 4700 1100
+Connection ~ 3000 2500
+Connection ~ 3000 2700
+Connection ~ 1800 2700
+Wire Wire Line
+	1800 2300 1800 3100
+Wire Wire Line
+	3000 3100 3000 2300
+Connection ~ 4500 1100
+Connection ~ 4500 2300
+Wire Wire Line
+	4100 2300 4900 2300
+Connection ~ 5700 3800
+Connection ~ 3300 2800
+Connection ~ 5300 2500
+Connection ~ 4150 3800
+Connection ~ 3800 2500
+Wire Wire Line
+	3800 2800 3800 2500
+Wire Wire Line
+	5300 2500 4300 2500
+Wire Wire Line
+	6600 3800 3800 3800
+Connection ~ 5750 4850
+Wire Wire Line
+	6450 5850 6450 4850
+Wire Wire Line
+	6450 4850 2150 4850
+Connection ~ 5250 7000
+Wire Wire Line
+	6450 6250 6450 7000
+Wire Wire Line
+	6450 7000 1800 7000
+Wire Wire Line
+	2850 5850 2850 6250
+Wire Wire Line
+	2650 6400 2650 6550
+Wire Wire Line
+	2650 6400 2450 6400
+Connection ~ 2450 7000
+Wire Wire Line
+	3250 6450 3250 6600
+Connection ~ 3250 4850
+Connection ~ 3800 4850
+Connection ~ 3800 7000
+Wire Wire Line
+	3800 7000 3800 7100
+Wire Wire Line
+	5750 5850 5750 6550
+Wire Wire Line
+	4850 6250 4950 6250
+Connection ~ 4300 5550
+Connection ~ 5050 5550
+Wire Wire Line
+	4500 5550 4300 5550
+Wire Wire Line
+	4500 5550 4850 5750
+Connection ~ 5050 5700
+Connection ~ 4300 5700
+Connection ~ 4100 7000
+Wire Wire Line
+	4100 7000 4100 6450
+Connection ~ 4300 4850
+Wire Wire Line
+	4300 4850 4300 5150
+Wire Wire Line
+	5750 6550 2650 6550
+Connection ~ 3250 7000
+Wire Wire Line
+	5400 3250 5700 3250
+Connection ~ 5950 3800
+Connection ~ 5700 3800
+Connection ~ 6100 1150
+Connection ~ 6200 2500
+Wire Wire Line
+	3000 2500 3300 2500
+Wire Wire Line
+	3300 2500 3300 2950
+Wire Wire Line
+	6100 2500 6100 2350
+Connection ~ 6100 2500
+Wire Wire Line
+	6550 3000 6200 3000
+Wire Wire Line
+	5700 2500 5700 2650
+Wire Wire Line
+	5300 2500 5300 2350
+Wire Wire Line
+	6200 2600 6200 2500
+Wire Wire Line
+	4700 2300 4700 2500
+Connection ~ 5600 1150
+Wire Wire Line
+	6200 3650 6200 3800
+Connection ~ 6200 3800
+Wire Wire Line
+	6200 3000 6200 3150
+Connection ~ 4700 2300
+Wire Wire Line
+	5400 2750 5400 2650
+Wire Wire Line
+	5400 2650 5700 2650
+Wire Wire Line
+	3250 5350 4000 5350
+Wire Wire Line
+	3250 5850 3250 6050
+Wire Wire Line
+	2150 5850 2150 6600
+Wire Wire Line
+	2150 4850 2150 5350
+Wire Wire Line
+	5050 4850 5050 5150
+Wire Wire Line
+	2150 6600 1800 6600
+Connection ~ 2150 6600
+Wire Wire Line
+	5250 7000 5250 6450
+Wire Wire Line
+	4300 5550 4300 5950
+Wire Wire Line
+	4300 5950 4100 5950
+Wire Wire Line
+	4100 5950 4100 6050
+Wire Wire Line
+	5050 5950 5050 5550
+Wire Wire Line
+	5050 5950 5250 5950
+Wire Wire Line
+	5250 5950 5250 6050
+Wire Wire Line
+	4500 5750 4850 5550
+Wire Wire Line
+	4850 5550 5050 5550
+Wire Wire Line
+	4400 6250 4500 6250
+Wire Wire Line
+	2850 6250 2950 6250
+Wire Wire Line
+	5350 5350 5750 5350
+Connection ~ 5050 4850
+Wire Wire Line
+	2450 6400 2450 6250
+Wire Wire Line
+	2450 6800 2450 7000
+Wire Wire Line
+	2850 5350 2850 4850
+Connection ~ 2850 4850
+Wire Wire Line
+	6100 7000 6100 6250
+Connection ~ 6100 7000
+Wire Wire Line
+	6100 4850 6100 5850
+Connection ~ 6100 4850
+Wire Wire Line
+	5100 950  5100 800
+Wire Wire Line
+	3300 3800 3300 3550
+Wire Wire Line
+	4300 2500 4300 2800
+Connection ~ 4300 2500
+Wire Wire Line
+	3900 2500 3700 2500
+Wire Wire Line
+	4100 1100 4900 1100
+Wire Wire Line
+	5700 3800 5700 3750
+Connection ~ 1800 2500
+Wire Wire Line
+	5600 1750 5300 1750
+Wire Wire Line
+	5300 1750 5300 1650
+Wire Wire Line
+	1800 7000 1800 6800
+Wire Wire Line
+	1650 2500 1800 2500
 Connection ~ 4700 2500
-Wire Wire Line
-	6600 1150 5300 1150
-Wire Wire Line
-	1650 2500 1800 2500
-Wire Wire Line
-	1800 6800 1800 7000
-Wire Wire Line
-	5300 1650 5300 1750
-Wire Wire Line
-	5300 1750 5600 1750
-Connection ~ 1800 2500
-Wire Wire Line
-	5700 3800 5700 3750
-Wire Wire Line
-	4100 1100 4900 1100
-Wire Wire Line
-	3900 2500 3700 2500
-Connection ~ 4300 2500
-Wire Wire Line
-	4300 2800 4300 2500
-Wire Wire Line
-	3300 3800 3300 3550
-Wire Wire Line
-	5100 950  5100 800
-Connection ~ 6100 4850
-Wire Wire Line
-	6100 4850 6100 5850
-Connection ~ 6100 7000
-Wire Wire Line
-	6100 7000 6100 6250
-Connection ~ 2850 4850
-Wire Wire Line
-	2850 5350 2850 4850
-Wire Wire Line
-	2450 6800 2450 7000
-Wire Wire Line
-	2450 6250 2450 6400
-Connection ~ 5050 4850
-Wire Wire Line
-	5350 5350 5750 5350
-Wire Wire Line
-	2950 6250 2850 6250
-Wire Wire Line
-	4400 6250 4500 6250
-Wire Wire Line
-	4850 5550 5050 5550
-Wire Wire Line
-	4850 5550 4500 5750
-Wire Wire Line
-	5250 6050 5250 5950
-Wire Wire Line
-	5250 5950 5050 5950
-Wire Wire Line
-	5050 5950 5050 5550
-Wire Wire Line
-	4100 6050 4100 5950
-Wire Wire Line
-	4100 5950 4300 5950
-Wire Wire Line
-	4300 5950 4300 5550
-Wire Wire Line
-	5250 7000 5250 6450
-Connection ~ 2150 6600
-Wire Wire Line
-	1800 6600 2150 6600
-Wire Wire Line
-	5050 4850 5050 5150
-Wire Wire Line
-	2150 5350 2150 4850
-Wire Wire Line
-	2150 6600 2150 5850
-Wire Wire Line
-	3250 5850 3250 6050
-Wire Wire Line
-	3250 5350 4000 5350
-Wire Wire Line
-	5400 2650 5700 2650
-Wire Wire Line
-	5400 2650 5400 2750
-Connection ~ 4700 2300
-Wire Wire Line
-	6200 3150 6200 3000
-Connection ~ 6200 3800
-Wire Wire Line
-	6200 3650 6200 3800
-Connection ~ 5600 1150
-Wire Wire Line
-	4700 2300 4700 2500
-Wire Wire Line
-	6200 2600 6200 2500
-Wire Wire Line
-	5300 2350 5300 2500
-Wire Wire Line
-	5700 2650 5700 2500
-Wire Wire Line
-	6200 3000 6550 3000
-Connection ~ 6100 2500
-Wire Wire Line
-	6100 2350 6100 2500
-Wire Wire Line
-	3300 2950 3300 2500
-Wire Wire Line
-	3300 2500 3000 2500
-Connection ~ 6200 2500
-Connection ~ 6100 1150
-Connection ~ 5700 3800
-Connection ~ 5950 3800
-Connection ~ 6400 1150
-Wire Wire Line
-	5400 3250 5700 3250
-Connection ~ 3250 7000
-Wire Wire Line
-	5750 6550 2650 6550
-Wire Wire Line
-	4300 4850 4300 5150
-Connection ~ 4300 4850
-Wire Wire Line
-	4100 7000 4100 6450
-Connection ~ 4100 7000
-Connection ~ 4300 5700
-Connection ~ 5050 5700
-Wire Wire Line
-	4850 5750 4500 5550
-Wire Wire Line
-	4500 5550 4300 5550
-Connection ~ 5050 5550
-Connection ~ 4300 5550
-Wire Wire Line
-	4850 6250 4950 6250
-Wire Wire Line
-	5750 6550 5750 5850
-Wire Wire Line
-	3800 7000 3800 7100
-Connection ~ 3800 7000
-Connection ~ 3800 4850
-Connection ~ 3250 4850
-Wire Wire Line
-	3250 6450 3250 6600
-Connection ~ 2450 7000
-Wire Wire Line
-	2450 6400 2650 6400
-Wire Wire Line
-	2650 6400 2650 6550
-Wire Wire Line
-	2850 6250 2850 5850
-Wire Wire Line
-	1800 7000 6450 7000
-Wire Wire Line
-	6450 7000 6450 6250
-Connection ~ 5250 7000
-Wire Wire Line
-	2150 4850 6450 4850
-Wire Wire Line
-	6450 4850 6450 5850
-Connection ~ 5750 4850
-Wire Wire Line
-	6600 3800 3800 3800
-Wire Wire Line
-	5300 2500 4300 2500
-Wire Wire Line
-	3800 2800 3800 2500
-Connection ~ 3800 2500
-Connection ~ 4150 3800
-Connection ~ 5300 2500
-Connection ~ 3300 2800
-Connection ~ 5700 3800
-Wire Wire Line
-	4100 2300 4900 2300
-Connection ~ 4500 2300
-Connection ~ 4500 1100
-Wire Wire Line
-	3000 3100 3000 2300
-Wire Wire Line
-	1800 2300 1800 3100
-Connection ~ 1800 2700
-Connection ~ 3000 2700
-Connection ~ 3000 2500
-Connection ~ 4700 1100
-Wire Wire Line
-	6100 2500 6400 2500
-Wire Wire Line
-	6400 1750 6100 1750
-Wire Wire Line
-	6100 1750 6100 1650
-Wire Wire Line
-	4700 950  4700 1100
-Wire Wire Line
-	6800 2500 6950 2500
-Connection ~ 3650 7000
-Connection ~ 3650 4850
-Connection ~ 5750 5350
-Connection ~ 3250 5350
-Connection ~ 3300 3800
-Connection ~ 3300 2500
-Connection ~ 6100 1750
-Connection ~ 5300 1750
-Connection ~ 11500 4850
 $Comp
 L CONN_1 Bias-2
@@
 $EndComp
 $Comp
-L GND #PWR016
-U 1 1 52CCC035
-P 6400 1550
-F 0 "#PWR016" H 6400 1550 30  0001 C CNN
-F 1 "GND" H 6400 1480 30  0001 C CNN
-	1    6400 1550
-	1    0    0    -1
-$EndComp
-$Comp
-L C C26
-U 1 1 52CCC028
-P 6400 1350
-F 0 "C26" H 6450 1450 50  0000 L CNN
-F 1 "0.1u" H 6450 1250 50  0000 L CNN
-	1    6400 1350
-	1    0    0    -1
-$EndComp
-$Comp
 L C C24
 U 1 1 52CCC014
@@
 $EndComp
 $Comp
-L GND #PWR017
+L GND #PWR016
 U 1 1 52CC826E
 P 6550 3400
-F 0 "#PWR017" H 6550 3400 30  0001 C CNN
+F 0 "#PWR016" H 6550 3400 30  0001 C CNN
 F 1 "GND" H 6550 3330 30  0001 C CNN
 	1    6550 3400
